File: pcb/EuroTap.kicad_sch (KiCad schematic)
At the start: 3 parts, among them J1 AudioJack3_Ground, J2 AudioJack3_Ground, J3 Conn_Coaxial

Commit message: 30cm width
Parts:
- J1, J2: footprint SloBlo:Jack_3.5mm_PJ311_Horizontal_Handsolder -> SloBlo:Jack_3.5mm_PJ311_Horizontal
Changed lines of the file:
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@@
 			)
 		)
-		(property "Footprint" "SloBlo:Jack_3.5mm_PJ311_Horizontal_Handsolder"
+		(property "Footprint" "SloBlo:Jack_3.5mm_PJ311_Horizontal"
 			(at 129.54 73.66 0)
 			(effects
@@
 			)
 		)
-		(property "Footprint" "SloBlo:Jack_3.5mm_PJ311_Horizontal_Handsolder"
+		(property "Footprint" "SloBlo:Jack_3.5mm_PJ311_Horizontal"
 			(at 129.54 99.06 0)
 			(effects
